File: Electrical/Circuit_Design_V1/Display.kicad_sch (KiCad schematic)
At the start: 18 parts, among them Q1 NMOS

Commit message: Completing schematic.
Parts:
- removed R4: 1650Ω, Resistor_SMD:R_0805_2012Metric, symbol Device:R
- removed R5: 1370Ω, Resistor_SMD:R_0805_2012Metric, symbol Device:R
- U3: footprint (none) -> Etchasketch_Footprints:F33Z-1A7Q1-E8C24
Connections:
- net +1V8: now reaches U3.18 (VDD)
- net +3.3V renamed +3V3
- net VPP: no longer names the net of U3.19 (VPP)
