File: electrical/display.kicad_sch (KiCad schematic)
At the start: 0 parts

Commit message: #3 Adding controls connections to STM32, updating IOC file to match.
Other:
- company: (none) -> AlumaPower
Changed lines of the file:
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@@
 	(generator_version "9.0")
 	(paper "A4")
+	(title_block
+		(company "AlumaPower")
+	)
 	(bus_entry
 		(at 55.88 59.69)

Commit message: #3 Updating schematic.
Parts:
- added C24, C25, C26, C27, C28, C29, C30, C31, C8: 1uF, SamacSys_Parts:MAJx16, symbol SamacSys_Parts:MAJCT168BB7105KTEA01
- added D1, D2, D3: ~, SamacSys_Parts:SOD3716X135N, symbol SamacSys_Parts:MBR0530T1G
- added J2: 687124149022, 687124149022, symbol SamacSys_Parts:687124149022
- added L1: 47uH, symbol Device:L
- added Q1: ~, SamacSys_Parts:SOT65P210X110-6N, symbol SamacSys_Parts:NX3008NBKS,115
- added R7: 2.2Ω, Resistor_SMD:R_0603_1608Metric_Pad0.98x0.95mm_HandSolder, symbol Device:R
- added R8: 1 kOhm, SamacSys_Parts:ERA3AEB101V, symbol SamacSys_Parts:ERA-3AED102V
- added R9: 1.5 kOhms, SamacSys_Parts:ERA3AEB101V, symbol SamacSys_Parts:ERA-3APB152V
Connections:
- net 3V0: now also C8.1, J2.15, J2.16, L1.2, R8.1
- new net: C29.1, D2.1 (K), D3.2 (A)
- new net: C29.2, D1.2 (A), L1.1, Q1.6 (D1)
- new net 1V8: C24.1, J2.18, R8.2, R9.1
- new net BS1: C24.2, C25.2, C26.2, C27.2, C28.2, C30.1, C31.1, C8.2, D3.1 (K), J2.17, J2.6, J2.7, J2.8, R9.2
- new net BUSY: J2.9
- new net CS: J2.12
- new net D/C#: J2.11
- new net GDR: J2.2, Q1.2 (G1), R7.2
- new net RES#: J2.10
- new net RESE: J2.3, Q1.1 (S1), R7.1
- new net SCL: J2.13
- new net SCREEN_SDA: J2.14
- new net VCOM: C27.1, J2.24
- new net VGH: C30.2, D1.1 (K), J2.21
- new net VGL: C31.2, D2.2 (A), J2.23
- new net VPP: J2.19
- new net VSH1: C25.1, J2.20
- new net VSH2: C28.1, J2.5
- new net VSL: C26.1, J2.22
- no-connect marks 0 -> 8

Commit message: #3 Finding CAD for switch.
Parts:
- removed L1: 47uH, symbol Device:L
- added L1: 47 uH, SamacSys_Parts:CDRH2D18LDNP470NC, symbol SamacSys_Parts:CDRH2D18_LDNP-470NC
Connections:
- net 3V0: now also L1.2
- net at C29.2, D1.2 (A), Q1.6 (D1): now also L1.1
Changed lines of the file:
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@@
 	(wire
 		(pts
-			(xy 151.13 97.79) (xy 161.29 97.79)
+			(xy 167.64 97.79) (xy 177.8 97.79)
 		)
 		(stroke
@@
 	(wire
 		(pts
-			(xy 143.51 97.79) (xy 138.43 97.79)
+			(xy 147.32 97.79) (xy 138.43 97.79)
 		)
 		(stroke
@@
 	)
 	(label "VCI"
-		(at 161.29 97.79 180)
+		(at 177.8 97.79 180)
 		(effects
 			(font
@@
 	)
 	(symbol
-		(lib_id "Device:L")
-		(at 147.32 97.79 90)
-		(unit 1)
-		(exclude_from_sim no)
-		(in_bom yes)
-		(on_board yes)
-		(dnp no)
-		(fields_autoplaced yes)
-		(property "Reference" "L1"
-			(at 147.32 92.71 90)
-			(effects
-				(font
-					(size 1.27 1.27)
-				)
-			)
-		)
-		(property "Value" "47uH"
-			(at 147.32 95.25 90)
-			(effects
-				(font
-					(size 1.27 1.27)
-				)
-			)
-		)
-		(property "Footprint" ""
-			(at 147.32 97.79 0)
-			(effects
-				(font
-					(size 1.27 1.27)
-				)
-				(hide yes)
-			)
-		)
-		(property "Datasheet" "https://products.sumida.com/products/pdf/CDRH2D18LD_Ver2.0_E.pdf"
-			(at 147.32 97.79 0)
-			(effects
-				(font
-					(size 1.27 1.27)
-				)
-				(hide yes)
-			)
-		)
-		(property "Description" "NOCAD"
-			(at 147.32 97.79 0)
-			(effects
-				(font
-					(size 1.27 1.27)
-				)
-			)
-		)
-		(pin "2"
-		)
-		(pin "1"
-		)
-		(instances
-			(project ""
-				(path "/0ea7de92-e138-4a6c-b193-fca6869c3a12/5c80e7a0-2fc8-469f-b7eb-810d0b40b08d"
-					(reference "L1")
-					(unit 1)
-				)
-			)
-		)
-	)
-	(symbol
 		(lib_id "SamacSys_Parts:MBR0530T1G")
 		(at 134.62 76.2 180)
@@
 					(unit 1)
 				)
+			)
+		)
+	)
+	(symbol
+		(lib_id "SamacSys_Parts:CDRH2D18_LDNP-470NC")
+		(at 147.32 97.79 0)
+		(unit 1)
+		(exclude_from_sim no)
+		(in_bom yes)
+		(on_board yes)
+		(dnp no)
+		(fields_autoplaced yes)
+		(property "Reference" "L1"
+			(at 157.48 91.44 0)
+			(effects
+				(font
+					(size 1.27 1.27)
+				)
+			)
+		)
+		(property "Value" "47 uH"
+			(at 157.48 93.98 0)
+			(effects
+				(font
+					(size 1.27 1.27)
+				)
+			)
+		)
+		(property "Footprint" "SamacSys_Parts:CDRH2D18LDNP470NC"
+			(at 163.83 193.98 0)
+			(effects
+				(font
+					(size 1.27 1.27)
+				)
+				(justify left top)
+				(hide yes)
+			)
+		)
+		(property "Datasheet" "https://products.sumida.com/products/pdf/CDRH2D18LD_Ver2.0_E.pdf"
+			(at 163.83 293.98 0)
+			(effects
+				(font
+					(size 1.27 1.27)
+				)
+				(justify left top)
+				(hide yes)
+			)
+		)
+		(property "Description" "47 H Shielded Inductor 480 mA 660mOhm Max Nonstandard -40C ~ 105C"
+			(at 147.32 97.79 0)
+			(effects
+				(font
+					(size 1.27 1.27)
+				)
+				(hide yes)
+			)
+		)
+		(property "Height" "2"
+			(at 163.83 493.98 0)
+			(effects
+				(font
+					(size 1.27 1.27)
+				)
+				(justify left top)
+				(hide yes)
+			)
+		)
+		(property "Mouser Part Number" "851-CDRH2D18LDNP470"
+			(at 163.83 593.98 0)
+			(effects
+				(font
+					(size 1.27 1.27)
+				)
+				(justify left top)
+				(hide yes)
+			)
+		)
+		(property "Mouser Price/Stock" "https://www.mouser.co.uk/ProductDetail/Sumida/CDRH2D18-LDNP-470NC?qs=mT6umqgwvA1P4peHEoEcxg%3D%3D"
+			(at 163.83 693.98 0)
+			(effects
+				(font
+					(size 1.27 1.27)
+				)
+				(justify left top)
+				(hide yes)
+			)
+		)
+		(property "Manufacturer_Name" "Sumida"
+			(at 163.83 793.98 0)
+			(effects
+				(font
+					(size 1.27 1.27)
+				)
+				(justify left top)
+				(hide yes)
+			)
+		)
+		(property "Manufacturer_Part_Number" "CDRH2D18/LDNP-470NC"
+			(at 163.83 893.98 0)
+			(effects
+				(font
+					(size 1.27 1.27)
+				)
+				(justify left top)
+				(hide yes)
+			)
+		)
+		(pin "1"
+		)
+		(pin "2"
+		)
+		(instances
+			(project ""
+				(path "/0ea7de92-e138-4a6c-b193-fca6869c3a12/5c80e7a0-2fc8-469f-b7eb-810d0b40b08d"
+					(reference "L1")
+					(unit 1)
+				)

Commit message: #17 Making layout. Errors rpesent.
Parts:
- J2: footprint 687124149022 -> SamacSys_Parts:687124149022
Connections:
- net BS1 renamed GND
- net BUSY renamed SCREEN_BUSY
- net CS renamed SCREEN_CS
- net D/C# renamed SCREEN_D_C
- net RES# renamed SCREEN_RST
- net SCL renamed SCREEN_SCL
- net VPP: no longer names the net of J2.19
