File: electrical/electrical.kicad_pcb (KiCad board)
At the start: 2 copper layers, 66 parts, among them IC1 STM32G484QET6, IC2 ADXL345BCCZ, J1 FTSH-107-01-F-DV-K, J2 687124149022, Y1 32.764KHz, Y3 24 MHz

Commit message: #17 Making layout. Errors rpesent.
Parts:
- removed R6: 10KΩ, SamacSys_Parts:RESC1608X58N
- added H5: MountingHole, MountingHole:MountingHole_2.2mm_M2, F.Cu at (171.9, 93.8)
- added H6: MountingHole, MountingHole:MountingHole_2.2mm_M2, F.Cu at (145.2, 93.8)
- BT1, C1, C24, C25, C26, C27, C28, C29, C3, C30, C31, C7, C8, D1, D2, D3, IC2, L1, LED1, Q1, R1, R3, R4, R7, R8, R9, S1, U1: moved to B.Cu
- moved R2 297.1 mm to (173.9, 105.7), turned to 90 degrees
- moved R4 277.3 mm to (181.1, 131.8), turned to -90 degrees
- moved IC2 275.9 mm to (184.6, 131.8), turned to 90 degrees
- moved FB1 275.2 mm to (184.2, 96.4)
- moved C3 274.9 mm to (186.6, 136.0), turned to -90 degrees
- moved C10 274.3 mm to (195.0, 76.0), turned to 180 degrees
- moved C7 270.5 mm to (182.6, 135.3), turned to -90 degrees
- moved Y1 264.0 mm to (166.5, 78.7), turned to 90 degrees
- moved C17 263.4 mm to (195.0, 82.4), turned to 180 degrees
- moved C13 261.2 mm to (187.5, 92.8), turned to 90 degrees
- moved C18 259.0 mm to (190.5, 92.8), turned to 90 degrees
- moved C14 258.9 mm to (184.6, 70.8), turned to -90 degrees
- moved C12 258.3 mm to (184.5, 92.8), turned to 90 degrees
- moved IC1 257.6 mm to (184.0, 81.8)
- moved C11 257.3 mm to (178.5, 92.8), turned to 90 degrees
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Connections:
- BT1 pad 1: +3V0 -> /Connectivity/3V0
- BT1 pad 2: GND -> /Connectivity/GND
- C1 pad 1: +3V0 -> /Connectivity/3V0
- C1 pad 2: GND -> /Connectivity/GND
- C10 pad 1: /Processor/GND -> /Connectivity/GND
- C10 pad 2: /Processor/3V0 -> /Connectivity/3V0
- C11 pad 1: /Processor/GND -> /Connectivity/GND
- C11 pad 2: /Processor/3V0 -> /Connectivity/3V0
- C12 pad 1: /Processor/GND -> /Connectivity/GND
- C12 pad 2: /Processor/3V0 -> /Connectivity/3V0
- C13 pad 1: /Processor/GND -> /Connectivity/GND
- C13 pad 2: /Processor/3V0 -> /Connectivity/3V0
- C14 pad 1: /Processor/GND -> /Connectivity/GND
- C14 pad 2: /Processor/3V0 -> /Connectivity/3V0
- C15 pad 1: /Processor/GND -> /Connectivity/GND
- C15 pad 2: /Processor/3V0 -> /Connectivity/3V0
- C16 pad 1: /Processor/GND -> /Connectivity/GND
- C16 pad 2: /Processor/3V0 -> /Connectivity/3V0
- C17 pad 1: /Processor/GND -> /Connectivity/GND
- C17 pad 2: /Processor/3V0 -> /Connectivity/3V0
- C18 pad 1: /Processor/GND -> /Connectivity/GND
- C18 pad 2: /Processor/3V0 -> /Connectivity/3V0
- C2 pad 1: /Processor/GND -> /Connectivity/GND
- C2 pad 2: /Processor/3V0 -> /Connectivity/3V0
- C20 pad 1: /Processor/GND -> /Connectivity/GND
- C20 pad 2: /Processor/3V0 -> /Connectivity/3V0
- C21 pad 1: /Processor/GND -> /Connectivity/GND
- C21 pad 2: /Processor/3V0 -> /Connectivity/3V0
- C22 pad 1: /Processor/GND -> /Connectivity/GND
- C24 pad 2: /Display/BS1 -> /Connectivity/GND
- C25 pad 2: /Display/BS1 -> /Connectivity/GND
- C26 pad 2: /Display/BS1 -> /Connectivity/GND
- C27 pad 2: /Display/BS1 -> /Connectivity/GND
- C28 pad 2: /Display/BS1 -> /Connectivity/GND
- C3 pad 1: /Controls/3V0 -> /Connectivity/3V0
- C3 pad 2: /Controls/GND -> /Connectivity/GND
- C30 pad 1: /Display/BS1 -> /Connectivity/GND
- C31 pad 1: /Display/BS1 -> /Connectivity/GND
- C32 pad 1: /Processor/GND -> /Connectivity/GND
- C33 pad 1: /Processor/GND -> /Connectivity/GND
- C4 pad 1: /Processor/3V0 -> /Connectivity/3V0
- C4 pad 2: /Processor/GND -> /Connectivity/GND
- C5 pad 2: /Processor/GND -> /Connectivity/GND
- C6 pad 1: /Processor/GND -> /Connectivity/GND
- C6 pad 2: /Processor/3V0 -> /Connectivity/3V0
- C7 pad 1: /Controls/3V0 -> /Connectivity/3V0
- C7 pad 2: /Controls/GND -> /Connectivity/GND
- C8 pad 1: /Display/3V0 -> /Connectivity/3V0
- C8 pad 2: /Display/BS1 -> /Connectivity/GND
- C9 pad 1: /Processor/GND -> /Connectivity/GND
- D3 pad 1: /Display/BS1 -> /Connectivity/GND
- FB1 pad 1: /Processor/3V0 -> /Connectivity/3V0
- FB1 pad 2: /Processor/3V0 -> /Connectivity/3V0
- IC1 pad 1: /Processor/SCREEN_SCL -> /Display/SCREEN_SCL
- IC1 pad 100: /Processor/WIFI_SCK -> /Connectivity/WIFI_SCK
- IC1 pad 101: /Processor/WIFI_MISO -> /Connectivity/WIFI_MISO
- IC1 pad 102: /Processor/WIFI_MOSI -> /Connectivity/WIFI_MOSI
- IC1 pad 103: /Processor/WIFI_BUSY -> /Connectivity/WIFI_BUSY
- IC1 pad 104: /Processor/WIFI_RESET -> /Connectivity/WIFI_RESET
- IC1 pad 110: /Processor/GND -> /Connectivity/GND
- IC1 pad 111: /Processor/3V0 -> /Connectivity/3V0
- IC1 pad 12: /Processor/GND -> /Connectivity/GND
- IC1 pad 127: /Processor/GND -> /Connectivity/GND
- IC1 pad 128: /Processor/3V0 -> /Connectivity/3V0
- IC1 pad 13: /Processor/3V0 -> /Connectivity/3V0
- IC1 pad 2: /Processor/SCREEN_BUSY -> /Display/SCREEN_BUSY
- IC1 pad 3: /Processor/SCREEN_CS -> /Display/SCREEN_CS
- IC1 pad 30: /Processor/GND -> /Connectivity/GND
- IC1 pad 31: /Processor/3V0 -> /Connectivity/3V0
- IC1 pad 4: /Processor/SCREEN_D_C -> /Display/SCREEN_D_C
- IC1 pad 42: /Processor/GND -> /Connectivity/GND
- IC1 pad 43: /Processor/3V0 -> /Connectivity/3V0
- IC1 pad 44: /Processor/3V0 -> /Connectivity/3V0
- IC1 pad 45: /Processor/3V0 -> /Connectivity/3V0
- IC1 pad 46: /Processor/GND -> /Connectivity/GND
- IC1 pad 47: /Processor/3V0 -> /Connectivity/3V0
- IC1 pad 5: /Processor/SCREEN_SDA -> /Display/SCREEN_SDA
- IC1 pad 6: /Processor/3V0 -> /Connectivity/3V0
- IC1 pad 63: /Processor/GND -> /Connectivity/GND
- IC1 pad 64: /Processor/3V0 -> /Connectivity/3V0
- IC1 pad 66: /Processor/ADXL_CS -> /Controls/ADXL_CS
- IC1 pad 67: /Processor/ADXL_SCL -> /Controls/ADXL_SCL
- IC1 pad 68: /Processor/ADXL_SDO -> /Controls/ADXL_SDO
- IC1 pad 69: /Processor/ADXL_SDI -> /Controls/ADXL_SDI
- IC1 pad 7: /Processor/SCREEN_RST -> /Display/SCREEN_RST
- IC1 pad 70: /Processor/ADXL_INT1 -> /Controls/ADXL_INT1
- IC1 pad 71: /Processor/ADXL_INT2 -> /Controls/ADXL_INT2
- IC1 pad 72: /Processor/BUTTON_1 -> /Controls/BUTTON_1
- IC1 pad 73: /Processor/BUTTON_2 -> /Controls/BUTTON_2
- IC1 pad 74: /Processor/POT_1 -> /Controls/POT_1
- IC1 pad 75: /Processor/POT_2 -> /Controls/POT_2
- IC1 pad 78: /Processor/GND -> /Connectivity/GND
- IC1 pad 79: /Processor/3V0 -> /Connectivity/3V0
- IC1 pad 94: /Processor/GND -> /Connectivity/GND
- IC1 pad 95: /Processor/3V0 -> /Connectivity/3V0
- IC1 pad 99: /Processor/WIFI_CS -> /Connectivity/WIFI_CS
- IC2 pad 1: /Controls/3V0 -> /Connectivity/3V0
- IC2 pad 11: /Controls/3V0 -> /Connectivity/3V0
- IC2 pad 2: /Controls/GND -> /Connectivity/GND
- IC2 pad 3: /Controls/3V0 -> /Connectivity/3V0
- IC2 pad 4: /Controls/GND -> /Connectivity/GND
- IC2 pad 5: /Controls/GND -> /Connectivity/GND
- IC2 pad 6: /Controls/3V0 -> /Connectivity/3V0
- J1 pad 03: /Processor/3V0 -> /Connectivity/3V0
- J1 pad 05: /Processor/GND -> /Connectivity/GND
- J1 pad 07: /Processor/GND -> /Connectivity/GND
- J1 pad 11: /Processor/GND -> /Connectivity/GND
- J2 pad 10: /Display/RES# -> /Display/SCREEN_RST
- J2 pad 11: /Display/D/C# -> /Display/SCREEN_D_C
- J2 pad 12: /Display/CS -> /Display/SCREEN_CS
- J2 pad 13: /Display/SCL -> /Display/SCREEN_SCL
- J2 pad 15: /Display/3V0 -> /Connectivity/3V0
- J2 pad 16: /Display/3V0 -> /Connectivity/3V0
- J2 pad 17: /Display/BS1 -> /Connectivity/GND
- J2 pad 19: /Display/VPP -> unconnected-(J2-Pad19)
- J2 pad 6: /Display/BS1 -> /Connectivity/GND
- J2 pad 7: /Display/BS1 -> /Connectivity/GND
- J2 pad 8: /Display/BS1 -> /Connectivity/GND
- J2 pad 9: /Display/BUSY -> /Display/SCREEN_BUSY
- L1 pad 2: /Display/3V0 -> /Connectivity/3V0
- LED1 pad 2: +3V0 -> /Connectivity/3V0
- R1 pad 1: GND -> /Connectivity/GND
- R2 pad 1: /Controls/3V0 -> /Connectivity/3V0
- R4 pad 1: /Controls/3V0 -> /Connectivity/3V0
- R5 pad 1: /Controls/3V0 -> /Connectivity/3V0
- R8 pad 1: /Display/3V0 -> /Connectivity/3V0
- R9 pad 2: /Display/BS1 -> /Connectivity/GND
- RV1 pad 2: /Controls/GND -> /Connectivity/GND
- RV1 pad 3: /Controls/3V0 -> /Connectivity/3V0
- RV2 pad 2: /Controls/GND -> /Connectivity/GND
- RV2 pad 3: /Controls/3V0 -> /Connectivity/3V0
- S1 pad A3: /Processor/3V0 -> /Connectivity/3V0
- S1 pad B3: /Processor/GND -> /Connectivity/GND
- S2 pad C1: /Controls/GND -> /Connectivity/GND
- S2 pad D1: /Controls/GND -> /Connectivity/GND
- S3 pad B1: /Controls/GND -> /Controls/BUTTON_2
- S3 pad C1: /Controls/BUTTON_2 -> /Connectivity/GND
- S3 pad D1: /Controls/GND -> /Connectivity/GND
- S4 pad C1: /Processor/GND -> /Connectivity/GND
- S4 pad D1: /Processor/GND -> /Connectivity/GND
- Y3 pad 2: /Processor/GND -> /Connectivity/GND
- Y3 pad 4: /Processor/GND -> /Connectivity/GND
Routing:
- net /Connectivity/3V0: track 0.00 -> 133.9 mm, vias 0 -> 17
- net /Controls/BUTTON_1: track 0.00 -> 107.5 mm
- net /Connectivity/GND: track 0.00 -> 106.5 mm, vias 0 -> 50
- net /Processor/SWDIO: track 0.00 -> 95.7 mm
- net /Processor/SWCLK: track 0.00 -> 91.6 mm
- net /Processor/NRST: track 0.00 -> 89.9 mm
- net /Controls/POT_1: track 0.00 -> 88.4 mm
- net /Display/SCREEN_SDA: track 0.00 -> 88.2 mm, vias 0 -> 2
- net /Display/SCREEN_SCL: track 0.00 -> 86.0 mm, vias 0 -> 2
- net /Display/SCREEN_RST: track 0.00 -> 83.9 mm, vias 0 -> 2
- net /Display/SCREEN_CS: track 0.00 -> 83.8 mm, vias 0 -> 2
- net /Display/SCREEN_D_C: track 0.00 -> 81.3 mm, vias 0 -> 2
- net /Controls/ADXL_SDI: track 0.00 -> 79.5 mm, vias 0 -> 1
- net /Display/SCREEN_BUSY: track 0.00 -> 76.8 mm, vias 0 -> 2
- net /Controls/ADXL_SCL: track 0.00 -> 75.3 mm, vias 0 -> 1
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- added copper zone on In2.Cu, net /Connectivity/3V0
- added copper zone on In1.Cu, net /Connectivity/GND
Other:
- board outline added: 85 x 90 mm
- copper layers 2 -> 4

Commit message: #17 Finish PCB layout.
Routing:
- net /Connectivity/3V0: track 133.9 -> 144.1 mm, vias 17 -> 24
- net /Controls/ADXL_CS: track 55.7 -> 61.8 mm
- net /Controls/POT_2: track 44.6 -> 50.6 mm
- net /Controls/POT_1: track 88.4 -> 94.4 mm
- net /Controls/ADXL_INT1: track 52.6 -> 58.0 mm
- net /Controls/ADXL_INT2: track 53.6 -> 58.7 mm
- net /Controls/ADXL_SDO: track 59.1 -> 63.9 mm
- net /Connectivity/GND: track 106.5 -> 105.3 mm
