File: electrical/electrical.kicad_pcb (KiCad board)
At the start: 2 copper layers, 84 x 89 mm, 57 parts, among them IC1 STM32G474CBT6TR, IC3 SMD_ADXL345BCCZ, J1 24 Pins, J2 6871XX149022_687124149022, Q1 SMD_MOSFET_NX3008NBKS, SW1 SMD_BUTTON, SW2 SMD_SWITCH_HORIZONTAL, SW3 SMD_BUTTON, SW4 SMD_BUTTON

Commit message: Adding more to layout.
Parts:
- removed J1: 24 Pins, adrians_favs:THT_CONNECTOR_JTAG_SWD
- BT2, C10, C11, IC2, IC3, R5, R7, R9, SW2: moved to B.Cu
- moved RV2 253.1 mm to (179.2, 126.5)
- moved SW4 231.9 mm to (173.0, 115.0)
- moved R6 230.1 mm to (151.0, 94.5), turned to 90 degrees
- moved IC2 220.0 mm to (155.2, 79.5)
- moved IC3 206.5 mm to (183.5, 117.5), turned to 90 degrees
- moved RV1 206.4 mm to (130.8, 126.5)
- moved C11 205.0 mm to (186.3, 120.5), turned to 180 degrees
- moved R9 203.3 mm to (179.8, 116.5), turned to -90 degrees
- moved R7 200.3 mm to (136.6, 108.0)
- moved C10 199.3 mm to (180.6, 120.5), turned to 180 degrees
- moved SW3 197.1 mm to (137.5, 115.0)
- moved SW1 196.2 mm to (155.0, 115.0)
- moved SW2 195.3 mm to (168.2, 107.0), turned to -90 degrees
- moved R5 189.7 mm to (161.8, 107.0)
- moved BT2 188.8 mm to (155.0, 128.5)
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Connections:
- IC1 pad 10: /Processor/BUTTON_1 -> unconnected-(IC1-PA2-Pad10)
- IC1 pad 25: unconnected-(IC1-PB11-Pad25) -> /Processor/BUTTON_1
- R5 pad 1: Net-(SW2A-B) -> /Processor/BOOT0
- R5 pad 2: /Processor/BOOT0 -> Net-(SW2A-B)
Routing:
- net /Processor/WIFI_BUSY: track 0.00 -> 84.2 mm, vias 0 -> 1
- net /Accelerometer/ADXL_SDI: track 0.00 -> 82.2 mm, vias 0 -> 1
- net /Processor/WIFI_CS: track 0.00 -> 79.5 mm, vias 0 -> 1
- net /Accelerometer/ADXL_SDO: track 0.00 -> 75.6 mm, vias 0 -> 2
- net /Accelerometer/ADXL_INT2: track 0.00 -> 67.8 mm
- net /Accelerometer/ADXL_INT1: track 0.00 -> 62.8 mm
- net /Processor/POT_1: track 0.00 -> 61.6 mm
- net /Processor/WIFI_RESET: track 0.00 -> 57.7 mm, vias 0 -> 1
- net /Accelerometer/ADXL_SCL: track 0.00 -> 54.3 mm
- net /Processor/WIFI_MOSI: track 0.00 -> 53.0 mm, vias 0 -> 1
- net /Processor/POT_2: track 0.00 -> 52.9 mm
- net /Processor/WIFI_MISO: track 0.00 -> 52.2 mm, vias 0 -> 1
- net /Processor/WIFI_SCK: track 0.00 -> 49.7 mm, vias 0 -> 1
- net /Accelerometer/ADXL_CS: track 0.00 -> 41.4 mm
- net /Processor/BUTTON_2: track 0.00 -> 30.0 mm, vias 0 -> 1
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Other:
- copper layers 2 -> 4

Commit message: Completing PCB layout.
Parts:
- removed H5, H6: MountingHole, MountingHole:MountingHole_2.2mm_M2
- added J1: 24 Pins, adrians_favs:THT_CONNECTOR_JTAG_SWD, F.Cu at (154.6, 128.2)
- C21, D1, R1, R10, R11, R2, R3, R4: moved to B.Cu
- moved R8 116.0 mm to (176.8, 110.0), turned to 180 degrees
- moved D1 114.4 mm to (178.3, 65.8)
- moved R1 106.5 mm to (174.3, 65.8)
- moved C18 92.1 mm to (143.9, 76.8)
- moved R2 78.0 mm to (166.3, 132.3), turned to -90 degrees
- moved C20 76.7 mm to (131.9, 91.2), turned to 180 degrees
- moved R3 76.4 mm to (163.3, 132.3), turned to 90 degrees
- moved L1 74.6 mm to (142.5, 84.2), turned to -90 degrees
- moved C14 74.2 mm to (132.3, 81.2), turned to 180 degrees
- moved C17 73.0 mm to (132.0, 89.8), turned to 180 degrees
- moved C19 72.9 mm to (131.8, 94.2)
- moved C16 72.4 mm to (132.1, 88.2), turned to 180 degrees
- moved C15 71.9 mm to (132.1, 86.8), turned to 180 degrees
- moved R4 68.5 mm to (155.8, 132.3), turned to 90 degrees
- moved C12 64.2 mm to (131.9, 92.8)
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Connections:
- C12 pad 1: GND -> /Screen/VSL
- C12 pad 2: /Screen/VSL -> GND
- C13 pad 1: GND -> /Screen/VCOM
- C13 pad 2: /Screen/VCOM -> GND
Routing:
- net /Processor/TDO: track 0.00 -> 95.1 mm, vias 0 -> 1
- net /Processor/TCK/SWCLK: track 0.00 -> 84.8 mm, vias 0 -> 1
- net /Processor/TMS/SWDAT: track 0.00 -> 79.2 mm, vias 0 -> 1
- net /Processor/TRST: track 0.00 -> 71.3 mm, vias 0 -> 1
- net /Processor/TDI: track 0.00 -> 69.9 mm, vias 0 -> 1
- net GND: track 21.3 -> 81.9 mm, vias 0 -> 27
- net /Screen/VGL: track 0.00 -> 45.7 mm
- net +3V0: track 26.4 -> 71.4 mm, vias 0 -> 20
- net /Processor/EINK_RST: track 0.00 -> 40.6 mm, vias 0 -> 1
- net /Accelerometer/ADXL_SCL: track 54.3 -> 92.1 mm, vias 0 -> 1
- net /Processor/EINK_BUSY: track 0.00 -> 31.7 mm, vias 0 -> 1
- net /Screen/VGH: track 0.00 -> 31.6 mm
- net /Processor/EINK_D_C: track 0.00 -> 31.3 mm, vias 0 -> 1
- net /Processor/EINK_CS: track 0.00 -> 30.4 mm, vias 0 -> 1
- net /Processor/NRST: track 27.7 -> 57.3 mm
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- added copper zone on In1.Cu, net +3V0
- added copper zone on In2.Cu, net GND
