File: electrical/electrical.kicad_pcb (KiCad board)
At the start: 4 copper layers, 84 x 89 mm, 55 parts, among them IC1 STM32G474CBT6TR, IC3 SMD_ADXL345BCCZ, J1 24 Pins, J2 6871XX149022_687124149022, Q1 SMD_MOSFET_NX3008NBKS, SW1 SMD_BUTTON, SW2 SMD_SWITCH_HORIZONTAL, SW3 SMD_BUTTON, SW4 SMD_BUTTON

Commit message: Adding build files.
Other:
- board text added: "AdrianTheHacker"
- board text added: "https://github.com/AdrianTheHacker/Etch-A-Sketch-Concept"

Commit message: Improving manufacturability of the board.
Parts:
- IC2: value ~ -> THT_WIFI_MODULE
Changed lines of the file:
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@@
 			(drillshape 0)
 			(scaleselection 1)
-			(outputdirectory "outputs/gerber/")
+			(outputdirectory "outputs/")
 		)
 	)
@@
 			)
 		)
-		(property "Value" "~"
+		(property "Value" "THT_WIFI_MODULE"
 			(at 0 -1 180)
 			(unlocked yes)
@@
 			)
 		)
-		(property "Store" "https://www.adafruit.com/product/4201"
+		(property "Supplier" "https://www.adafruit.com/product/4201"
 			(at 0 0 180)
 			(unlocked yes)
@@
 		(sheetname "/WiFi/")
 		(sheetfile "wifi.kicad_sch")
-		(attr smd)
+		(attr smd dnp)
 		(fp_rect
 			(start -16 16.5)
