File: electrical/accelerometer.kicad_sch (KiCad schematic)
At the start: 0 parts

Commit message: Completing schematic.
Parts:
- added C10: 1UF, adrians_favs:SMD_CAPACITOR_TANTALUM_0603_1UF, symbol adrians_favs:SMD_CAPACITOR_TANTALUM_0603_1UF
- added C11: 100NF, adrians_favs:SMD_CAPACITOR_CERAMIC_0603, symbol adrians_favs:SMD_CAPACITOR_CERAMIC_0603_100NF
- added IC3: SMD_ADXL345BCCZ, adrians_favs:SMD_ADXL345BCCZ, symbol adrians_favs:SMD_ADXL345BCCZ
- added R9: 10KR, adrians_favs:SMD_RESISTOR_0603, symbol adrians_favs:SMD_RESISTOR_0603_10KR
Connections:
- new net +3V0: C10.2, C11.1, IC3.1 (VDD_I/O), IC3.11 (RESERVED), IC3.3 (RESERVED_2), IC3.6 (VS), R9.1
- new net ADXL_CS: IC3.7 (~{CS}), R9.2
- new net ADXL_INT1: IC3.8 (INT1)
- new net ADXL_INT2: IC3.9 (INT2)
- new net ADXL_SCL: IC3.14 (SCL/SCLK)
- new net ADXL_SDI: IC3.13 (SDA/SDI/SDIO)
- new net ADXL_SDO: IC3.12 (SDO/ALT_ADDRESS)
- new net GND: C10.1, C11.2, IC3.2 (GND_2), IC3.4 (GND_3), IC3.5 (GND)

Commit message: Adding manufacturer and manufacturer number to path.
Parts:
- C10: MFG (none) -> KYOCERA AVX; MFG P/N (none) -> TACL105K010FTA
- C11: MFG (none) -> KYOCERA AVX; MFG P/N (none) -> 06031C104MAT2A
- IC3: MFG (none) -> Analog Devices; MFG P/N (none) -> ADXL345BCCZ
- R9: MFG (none) -> Vishay / Draloric; MFG P/N (none) -> RCA060310K0JNEA
Changed lines of the file:
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@@
+			)
+		)
+		(property "MFG" "KYOCERA AVX"
+			(at 127 63.5 0)
+			(effects
+				(font
+					(size 1.27 1.27)
+				)
+				(hide yes)
+			)
+		)
+		(property "MFG P/N" "06031C104MAT2A"
+			(at 127 63.5 0)
+			(effects
+				(font
+					(size 1.27 1.27)
+				)
+				(hide yes)
+			)
+		)
+		(property "https://mou.sr/3MG6oNW" ""
+			(at 127 63.5 0)
+			(effects
+				(font
+					(size 1.27 1.27)
+				)
+				(hide yes)
 			)
 		)
@@
 			)
 		)
+		(property "MFG" "KYOCERA AVX"
+			(at 109.22 82.55 0)
+			(effects
+				(font
+					(size 1.27 1.27)
+				)
+				(hide yes)
+			)
+		)
+		(property "MFG P/N" "TACL105K010FTA"
+			(at 109.22 82.55 0)
+			(effects
+				(font
+					(size 1.27 1.27)
+				)
+				(hide yes)
+			)
+		)
+		(property "https://mou.sr/3MG6oNW" ""
+			(at 109.22 82.55 0)
+			(effects
+				(font
+					(size 1.27 1.27)
+				)
+				(hide yes)
+			)
+		)
 		(pin "1"
 		)
@@
 			)
 		)
+		(property "MFG" "Analog Devices"
+			(at 157.48 81.28 0)
+			(effects
+				(font
+					(size 1.27 1.27)
+				)
+				(hide yes)
+			)
+		)
+		(property "MFG P/N" "ADXL345BCCZ"
+			(at 157.48 81.28 0)
+			(effects
+				(font
+					(size 1.27 1.27)
+				)
+				(hide yes)
+			)
+		)
+		(property "https://mou.sr/3MG6oNW" ""
+			(at 157.48 81.28 0)
+			(effects
+				(font
+					(size 1.27 1.27)
+				)
+				(hide yes)
+			)
+		)
 		(pin "3"
 		)
@@
 			(effects
 				(font
+					(size 1.27 1.27)
+				)
+				(hide yes)
+			)
+		)
+		(property "MFG" "Vishay / Draloric"
+			(at 127 92.71 90)
+			(effects
+				(font
+					(size 1.27 1.27)
+				)
+				(hide yes)
+			)
+		)
+		(property "MFG P/N" "RCA060310K0JNEA"
+			(at 127 92.71 90)
+			(effects
+				(font
+					(size 1.27 1.27)
+				)
+				(hide yes)
+			)
+		)
+		(property "https://mou.sr/3MG6oNW" ""
+			(at 127 92.71 90)
+			(effects
+				(font

Commit message: Updating schematic pages.
Other:
- company: (none) -> github.com/AdrianTheHacker
- title: (none) -> Etchasketch Accelerometer
Changed lines of the file:
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@@
 	(generator_version "9.0")
 	(paper "A4")
+	(title_block
+		(title "Etchasketch Accelerometer")
+		(rev "2.0")
+		(company "github.com/AdrianTheHacker")
+	)
 	(bus_alias "ADXL_INTERFACE"
 		(members "ADXL_INT1" "ADXL_INT2" "ADXL_CS" "ADXL_SCL" "ADXL_SDO" "ADXL_SDI")
