File: electrical/power.kicad_sch (KiCad schematic)
At the start: 4 parts

Commit message: Adding manufacturer and manufacturer number to path.
Parts:
- BT2: MFG (none) -> Renata; MFG P/N (none) -> SMTU2032-G.TR
- C21: MFG (none) -> KYOCERA AVX; MFG P/N (none) -> 06034D106KAT2A
- D1: MFG (none) -> ams OSRAM; MFG P/N (none) -> KT EELP41.12-S2U1-25-2X4X-5-R18; Store (none) -> https://mou.sr/3MG6oNW; https://mou.sr/3MG6oNW https://mou.sr/3MG6oNW -> (none)
- R1: MFG (none) -> TE Connectivity / Holsworthy; MFG P/N (none) -> RT73F1J110RBTD
Changed lines of the file:
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@@
+			)
+		)
+		(property "MFG" "KYOCERA AVX"
+			(at 124.46 95.25 90)
+			(effects
+				(font
+					(size 1.27 1.27)
+				)
+				(hide yes)
+			)
+		)
+		(property "MFG P/N" "06034D106KAT2A"
+			(at 124.46 95.25 90)
+			(effects
+				(font
+					(size 1.27 1.27)
+				)
+				(hide yes)
+			)
+		)
+		(property "https://mou.sr/3MG6oNW" ""
+			(at 124.46 95.25 90)
+			(effects
+				(font
+					(size 1.27 1.27)
+				)
+				(hide yes)
 			)
 		)
@@
 			)
 		)
+		(property "MFG" "Renata"
+			(at 124.46 74.93 0)
+			(effects
+				(font
+					(size 1.27 1.27)
+				)
+				(hide yes)
+			)
+		)
+		(property "MFG P/N" "SMTU2032-G.TR"
+			(at 124.46 74.93 0)
+			(effects
+				(font
+					(size 1.27 1.27)
+				)
+				(hide yes)
+			)
+		)
+		(property "https://mou.sr/3MG6oNW" ""
+			(at 124.46 74.93 0)
+			(effects
+				(font
+					(size 1.27 1.27)
+				)
+				(hide yes)
+			)
+		)
 		(pin "2"
 		)
@@
 			)
 		)
+		(property "MFG" "TE Connectivity / Holsworthy"
+			(at 149.86 90.17 90)
+			(effects
+				(font
+					(size 1.27 1.27)
+				)
+				(hide yes)
+			)
+		)
+		(property "MFG P/N" "RT73F1J110RBTD"
+			(at 149.86 90.17 90)
+			(effects
+				(font
+					(size 1.27 1.27)
+				)
+				(hide yes)
+			)
+		)
+		(property "https://mou.sr/3MG6oNW" ""
+			(at 149.86 90.17 90)
+			(effects
+				(font
+					(size 1.27 1.27)
+				)
+				(hide yes)
+			)
+		)
 		(pin "2"
 		)
@@
 			)
 		)
-		(property "Datasheet" "https://look.ams-osram.com/m/4cbb1524123e38e9/original/KT-EELP41-12.pdf"
+		(property "Datasheet" "~"
 			(at 149.86 80.17 0)
 			(effects
@@
 			)
 		)
-		(property "https://mou.sr/3MG6oNW" "https://mou.sr/3MG6oNW"
+		(property "Store" "https://mou.sr/3MG6oNW"
 			(at 149.86 80.17 0)
 			(effects
 				(font
+					(size 1.27 1.27)
+				)
+				(hide yes)
+			)
+		)
+		(property "MFG" "ams OSRAM"
+			(at 149.86 80.17 90)
+			(effects
+				(font
+					(size 1.27 1.27)
+				)
+				(hide yes)
+			)
+		)
+		(property "MFG P/N" "KT EELP41.12-S2U1-25-2X4X-5-R18"
+			(at 149.86 80.17 90)
+			(effects
+				(font
+					(size 1.27 1.27)
+				)
+				(hide yes)
+			)
+		)
+		(property "https://mou.sr/3MG6oNW" ""
+			(at 149.86 80.17 90)
+			(effects
+				(font

Commit message: Updating schematic pages.
Other:
- company: (none) -> github.com/AdrianTheHacker
- title: (none) -> Etchasketch Power
Changed lines of the file:
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@@
 	(generator_version "9.0")
 	(paper "A4")
+	(title_block
+		(title "Etchasketch Power")
+		(date "2025-12-08")
+		(rev "2.0")
+		(company "github.com/AdrianTheHacker")
+	)
 	(junction
 		(at 115.57 95.25)
