File: electrical/processor.kicad_sch (KiCad schematic)
At the start: 28 parts, among them IC1 STM32G484QET6, J1 FTSH-107-01-F-DV-K, Y1 32.764KHz, Y3 24 MHz

Commit message: Making progress on schematic and developing IOC.
Parts:
- removed C10, C11, C12, C13, C14, C15, C16, C17, C18, C20, C21, C5: 100nF, SamacSys_Parts:MAJx16, symbol SamacSys_Parts:MAJCH168BB7104KTEA01
- removed C2, C6: 1uF, SamacSys_Parts:MAJx16, symbol SamacSys_Parts:MAJCT168BB7105KTEA01
- removed C22, C9: 6.8pF, SamacSys_Parts:CAPC1608X90N, symbol SamacSys_Parts:0603YA6R8CAT2A
- removed C32, C33: 20pF, SamacSys_Parts:CAPC1608X90N, symbol SamacSys_Parts:06031A200KAT2A
- removed C4: 10nF, SamacSys_Parts:CAPC1608X90N, symbol SamacSys_Parts:06035A103JAT2A
- removed FB1: ~, SamacSys_Parts:BMCQ1E0000H, symbol SamacSys_Parts:BMC-Q1E0000H
- removed IC1: STM32G484QET6, SamacSys_Parts:QFP40P1600X1600X160-128N, symbol SamacSys_Parts:STM32G484QET6
- removed J1: FTSH-107-01-F-DV-K, FTSH-107-01-F-DV-K:SAMTEC_FTSH-107-01-F-DV-K, symbol FTSH-107-01-F-DV-K:FTSH-107-01-F-DV-K
- removed R10: 390Ω, SamacSys_Parts:RESC1608X58N, symbol SamacSys_Parts:MCT0603MD3900BP500
- removed R3: 10KΩ, SamacSys_Parts:RESC1608X58N, symbol SamacSys_Parts:RA73F1J10KBTDF
- removed S1: MHSS1104, SamacSys_Parts:MHSS1104, symbol SamacSys_Parts:MHSS1104
- removed S4: PTS125SM73SMTR21M_LFS, SamacSys_Parts:PTS125SM73SMTR21MLFS, symbol SamacSys_Parts:PTS125SM73SMTR21M_LFS
- removed Y1: 32.764KHz, SamacSys_Parts:XT1312HHRXX32K76E, symbol SamacSys_Parts:XT1312HHRXX32K76E
- removed Y3: 24 MHz, SamacSys_Parts:CX3225FB24000C0FZZH1, symbol SamacSys_Parts:CX3225FB24000C0FZZH1
- added C1, C2, C3, C5, C7, C9: 100NF, adrians_favs:SMD_CAPACITOR_CERAMIC_0603, symbol adrians_favs:SMD_CAPACITOR_CERAMIC_0603_100NF
- added C4: 10UF, adrians_favs:SMD_CAPACITOR_CERAMIC_0603, symbol adrians_favs:SMD_CAPACITOR_CERAMIC_0603_10UF
- added C6, C8: 1UF, adrians_favs:SMD_CAPACITOR_CERAMIC_0603, symbol adrians_favs:SMD_CAPACITOR_CERAMIC_0603_1UF
- added IC1: STM32G474CBT6TR, adrians_favs:SMD_STM32G474CBT6TR, symbol adrians_favs:SMD_STM32G474CBT6TR
- added J1: 24 Pins, adrians_favs:THT_CONNECTOR_JTAG_SWD, symbol adrians_favs:THT_CONNECTOR_JTAG_SWD
- added R2, R3, R4, R5: 10KR, adrians_favs:SMD_RESISTOR_0603, symbol adrians_favs:SMD_RESISTOR_0603_10KR
- added SW1: SMD_BUTTON, adrians_favs:SMD_BUTTON, symbol adrians_favs:SMD_BUTTON
- added SW2: SMD_SWITCH_HORIZONTAL, adrians_favs:SMD_SWITCH_HORIZONTAL, symbol adrians_favs:SMD_SWITCH_HORIZONTAL
Connections:
- net BOOT0: now also IC1.45 (PB8-BOOT0), R5.2
- net GND: now also C1.1, C2.1, C3.1, C4.2, C5.1, C6.2, C7.1, C8.2, C9.2, IC1.19 (VSSA), IC1.23 (VSS_1), IC1.35 (VSS_2), IC1.47 (VSS_3), J1.10, J1.12, J1.14, J1.16, J1.18, J1.20, J1.4, J1.6, J1.8, R2.2, R3.1, R4.1, SW1.1, SW1.2, SW2.3 (C)
- net NRST: now also C9.1, IC1.7 (PG10_-_NRST), J1.15, SW1.3 (K), SW1.4 (A)
- net WIFI_BUSY: now also IC1.17 (PB1)
- net WIFI_CS: now also IC1.12 (PA4)
- net WIFI_MISO: now also IC1.14 (PA6)
- net WIFI_MOSI: now also IC1.15 (PA7)
- net WIFI_RESET: now also IC1.16 (PB0)
- net WIFI_SCK: now also IC1.13 (PA5)
- new net: J1.11, R4.2
- new net: J1.17, R3.2
- new net: R5.1, SW2.2 (B)
- new net: J1.19, R2.1
- new net +3V0: C1.2, C2.2, C3.2, C4.1, C5.2, C6.1, C7.2, C8.1, IC1.1 (VBAT), IC1.20 (VREF+), IC1.21 (VDDA), IC1.24 (VDD_1), IC1.36 (VDD_2), IC1.48 (VDD_3), J1.1, J1.2, SW2.1 (A)
- new net TCK/SWCLK: IC1.38 (PA14), J1.9
- new net TDI: IC1.39 (PA15), J1.5
- new net TDO: IC1.40 (PB3), J1.13
- new net TMS/SWDAT: IC1.37 (PA13), J1.7
- new net TRST: IC1.41 (PB4), J1.3
- no-connect marks 80 -> 25
Other:
- note added: "Decoupling for VDDA"
- note added: "Decoupling for VDD_1, VDD_2, VDD_3"
- note added: "Decoupling for VREF"
- note added: "Reset"
- note removed: "Oscillators"
- note removed: "VDD/VBAT/VREF+ Decoupling"
- company: AlumaPower -> (none)
- title: Etchasketch - Processor -> (none)

Commit message: Adding user input.
Connections:
- net BUTTON_1: now reaches IC1.10 (PA2)
- net BUTTON_2: now reaches IC1.4 (PC15_-_OSC32_OUT)
- net POT_2: now reaches IC1.8 (PA0)
- net POT_1: now reaches IC1.9 (PA1)
- no-connect marks 25 -> 21
Changed lines of the file:
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@@
-	)
-	(no_connect
-		(at 222.25 139.7)
 	)
 	(no_connect
@@
 	)
 	(no_connect
-		(at 209.55 139.7)
-	)
-	(no_connect
 		(at 247.65 109.22)
 	)
@@
 	)
 	(no_connect
-		(at 219.71 139.7)
-	)
-	(no_connect
 		(at 212.09 139.7)
 	)
@@
 	(no_connect
 		(at 179.07 121.92)
-	)
-	(no_connect
-		(at 224.79 139.7)
 	)
 	(no_connect
@@
 	)
 	(bus_entry
+		(at 161.29 43.18)
+		(size 2.54 2.54)
+		(stroke
+			(width 0)
+			(type default)
+		)
+	)
+	(bus_entry
+		(at 157.48 43.18)
+		(size 2.54 2.54)
+		(stroke
+			(width 0)
+			(type default)
+		)
+	)
+	(bus_entry
 		(at 179.07 24.13)
+		(size 2.54 2.54)
+		(stroke
+			(width 0)
+			(type default)
+		)
+	)
+	(bus_entry
+		(at 168.91 43.18)
 		(size 2.54 2.54)
 		(stroke
@@
 	)
 	(bus_entry
+		(at 165.1 43.18)
+		(size 2.54 2.54)
+		(stroke
+			(width 0)
+			(type default)
+		)
+	)
+	(bus_entry
 		(at 166.37 24.13)
 		(size 2.54 2.54)
@@
 	(wire
 		(pts
+			(xy 219.71 139.7) (xy 219.71 151.13)
+		)
+		(stroke
+			(width 0)
+			(type default)
+		)
+	)
+	(wire
+		(pts
 			(xy 92.71 166.37) (xy 104.14 166.37)
 		)
@@
 	(wire
 		(pts
+			(xy 222.25 139.7) (xy 222.25 151.13)
+		)
+		(stroke
+			(width 0)
+			(type default)
+		)
+	)
+	(bus
+		(pts
+			(xy 165.1 43.18) (xy 168.91 43.18)
+		)
+		(stroke
+			(width 0)
+			(type default)
+		)
+	)
+	(wire
+		(pts
 			(xy 166.37 124.46) (xy 179.07 124.46)
 		)
@@
 		)
 	)
+	(wire
+		(pts
+			(xy 163.83 45.72) (xy 163.83 59.69)
+		)
+		(stroke
+			(width 0)
+			(type default)
+		)
+	)
 	(bus
 		(pts
@@
 		)
 	)
+	(wire
+		(pts
+			(xy 167.64 45.72) (xy 167.64 59.69)
+		)
+		(stroke
+			(width 0)
+			(type default)
+		)
+	)
 	(polyline
 		(pts
@@
 	(wire
 		(pts
+			(xy 209.55 139.7) (xy 209.55 151.13)
+		)
+		(stroke
+			(width 0)
+			(type default)
+		)
+	)
+	(wire
+		(pts
 			(xy 39.37 78.74) (xy 39.37 76.2)
 		)
@@
 		)
 	)
+	(bus
+		(pts
+			(xy 161.29 43.18) (xy 165.1 43.18)
+		)
+		(stroke
+			(width 0)
+			(type default)
+		)
+	)
 	(wire
 		(pts
@@
 	(wire
 		(pts
+			(xy 224.79 139.7) (xy 224.79 151.13)
+		)
+		(stroke
+			(width 0)
+			(type default)
+		)
+	)
+	(wire
+		(pts
+			(xy 171.45 45.72) (xy 171.45 59.69)
+		)
+		(stroke
+			(width 0)
+			(type default)
+		)
+	)
+	(wire
+		(pts
 			(xy 74.93 86.36) (xy 91.44 86.36)
 		)
@@
 		)
 	)
+	(bus
+		(pts
+			(xy 157.48 43.18) (xy 161.29 43.18)
+		)
+		(stroke
+			(width 0)
+			(type default)
+		)
+	)
 	(wire
 		(pts
@@
 	(wire
 		(pts
+			(xy 160.02 45.72) (xy 160.02 59.69)
+		)
+		(stroke
+			(width 0)
+			(type default)
+		)
+	)
+	(wire
+		(pts
 			(xy 55.88 153.67) (xy 68.58 153.67)
+		)
+		(stroke
+			(width 0)
+			(type default)
+		)
+	)
+	(bus
+		(pts
+			(xy 153.67 43.18) (xy 157.48 43.18)
 		)
 		(stroke
@@
 		)
 	)
+	(label "POT_2"
+		(at 160.02 59.69 90)
+		(effects
+			(font
+				(size 1.27 1.27)
+			)
+			(justify left bottom)
+		)
+	)
 	(label "WIFI_RESET"
 		(at 162.56 38.1 90)
@@
 		)
 	)
+	(label "POT_1"
+		(at 222.25 151.13 90)
+		(effects
+			(font
+				(size 1.27 1.27)
+			)
+			(justify left bottom)
+		)
+	)
 	(label "WIFI_RESET"
 		(at 260.35 124.46 180)
@@
 		)
 	)
+	(label "BUTTON_1"
+		(at 224.79 151.13 90)
+		(effects
+			(font
+				(size 1.27 1.27)
+			)
+			(justify left bottom)
+		)
+	)
 	(label "TDO"
 		(at 166.37 111.76 0)
@@
 		)
 	)
+	(label "POT_1"
+		(at 163.83 59.69 90)
+		(effects
+			(font
+				(size 1.27 1.27)
+			)
+			(justify left bottom)
+		)
+	)
 	(label "WIFI_CS"
 		(at 229.87 151.13 90)
@@
 		)
 	)
+	(label "BUTTON_1"
+		(at 171.45 59.69 90)
+		(effects
+			(font
+				(size 1.27 1.27)
+			)
+			(justify left bottom)
+		)
+	)
 	(label "WIFI_BUSY"
 		(at 168.91 38.1 90)
@@
 		)
 	)
+	(label "POT_2"
+		(at 219.71 151.13 90)
+		(effects
+			(font
+				(size 1.27 1.27)
+			)
+			(justify left bottom)
+		)
+	)
+	(label "BUTTON_2"
+		(at 167.64 59.69 90)
+		(effects
+			(font
+				(size 1.27 1.27)
+			)
+			(justify left bottom)
+		)
+	)
 	(label "TDI"
 		(at 87.63 93.98 180)
@@
 		)
 	)
+	(label "BUTTON_2"
+		(at 209.55 151.13 90)
+		(effects
+			(font
+				(size 1.27 1.27)
+			)
+			(justify left bottom)
+		)
+	)
 	(label "TMS{slash}SWDAT"
 		(at 87.63 91.44 180)
@@
 	)
 	(global_label "+3V0"
-		(shape input)
+		(shape passive)
 		(at 252.73 30.48 180)
 		(fields_autoplaced yes)
@@
 		)
 		(property "Intersheetrefs" "${INTERSHEET_REFS}"
-			(at 244.6648 30.48 0)
+			(at 245.7761 30.48 0)
 			(effects
 				(font
@@
 	)
 	(global_label "GND"
-		(shape input)
+		(shape passive)
 		(at 252.73 24.13 180)
 		(fields_autoplaced yes)
@@
 		)
 		(property "Intersheetrefs" "${INTERSHEET_REFS}"
-			(at 245.8743 24.13 0)
+			(at 246.9856 24.13 0)
 			(effects
 				(font
@@
 		)
 	)
+	(hierarchical_label "{USER_INPUTS}"
+		(shape passive)
+		(at 153.67 43.18 180)
+		(effects
+			(font
+				(size 1.27 1.27)
+			)
+			(justify right)
+		)
+	)

Commit message: Completing schematic.
Connections:
- net EINK_RST: now reaches IC1.30 (PA8)
- net ADXL_INT1: now reaches IC1.31 (PA9)
- net ADXL_SDO: now reaches IC1.32 (PA10)
- net ADXL_SDI: now reaches IC1.33 (PA11)
- net ADXL_INT2: now reaches IC1.34 (PA12)
- net EINK_CS: now reaches IC1.42 (PB5)
- net EINK_BUSY: now reaches IC1.43 (PB6)
- net EINK_D_C: now reaches IC1.44 (PB7)
- net ADXL_CS: now reaches IC1.5 (PF0_-_OSC_IN)
- net ADXL_SCL: now reaches IC1.6 (PF1_-_OSC_OUT)
- no-connect marks 21 -> 11

Commit message: Adding more to layout.
Connections:
- net BOOT0: now also R5.1; no longer R5.2
- net BUTTON_1: now also IC1.25 (PB11); no longer IC1.10 (PA2)
- net at SW2.2 (B): now also R5.2; no longer R5.1
Changed lines of the file:
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@@
 	)
 	(no_connect
-		(at 179.07 127)
+		(at 224.79 139.7)
 	)
 	(no_connect
-		(at 222.25 93.98)
+		(at 179.07 127)
 	)
 	(no_connect
-		(at 229.87 93.98)
+		(at 222.25 93.98)
 	)
 	(bus_entry
@@
 	(wire
 		(pts
-			(xy 224.79 139.7) (xy 224.79 151.13)
-		)
-		(stroke
-			(width 0)
-			(type default)
-		)
-	)
-	(wire
-		(pts
 			(xy 171.45 45.72) (xy 171.45 59.69)
 		)
@@
 	(wire
 		(pts
+			(xy 229.87 82.55) (xy 229.87 93.98)
+		)
+		(stroke
+			(width 0)
+			(type default)
+		)
+	)
+	(wire
+		(pts
 			(xy 39.37 78.74) (xy 52.07 78.74)
 		)
@@
 		)
 	)
+	(label "BUTTON_1"
+		(at 229.87 82.55 270)
+		(effects
+			(font
+				(size 1.27 1.27)
+			)
+			(justify right bottom)
+		)
+	)
 	(label "WIFI_RESET"
 		(at 162.56 38.1 90)
@@
 		)
 	)
-	(label "BUTTON_1"
-		(at 224.79 151.13 90)
-		(effects
-			(font
-				(size 1.27 1.27)
-			)
-			(justify left bottom)
-		)
-	)
 	(label "ADXL_SDO"
 		(at 257.81 38.1 90)
@@
 		(lib_id "adrians_favs:SMD_RESISTOR_0603_10KR")
 		(at 105.41 41.91 0)
+		(mirror y)
 		(unit 1)
 		(exclude_from_sim no)
@@
 		(on_board yes)
 		(dnp no)
-		(fields_autoplaced yes)
 		(property "Reference" "R5"
 			(at 105.41 35.56 0)

Commit message: Adding manufacturer and manufacturer number to path.
Parts:
- C1, C2, C3, C5, C7, C9: MFG (none) -> KYOCERA AVX; MFG P/N (none) -> 06031C104MAT2A
- C4: MFG (none) -> KYOCERA AVX; MFG P/N (none) -> 06034D106KAT2A
- C6, C8: MFG (none) -> KYOCERA AVX; MFG P/N (none) -> 0603DC105MAT2A
- IC1: MFG (none) -> STMicroelectronics; MFG P/N (none) -> STM32G474CBT6TR
- J1: MFG (none) -> TE Connectivity; MFG P/N (none) -> 103308-5
- R2, R3, R4, R5: MFG (none) -> Vishay / Draloric; MFG P/N (none) -> RCA060310K0JNEA
- SW1: MFG (none) -> E-Switch; MFG P/N (none) -> TL3301CF260QG; Store (none) -> https://mou.sr/3MCeAPf
- SW2: MFG (none) -> C&K; MFG P/N (none) -> AYZ0102AGRLC

Commit message: Updating schematic pages.
Other:
- company: (none) -> github.com/AdrianTheHacker
- title: (none) -> Etchasketch Processor
Changed lines of the file:
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@@
 	(generator_version "9.0")
 	(paper "A4")
+	(title_block
+		(title "Etchasketch Processor")
+		(date "2025-11-12")
+		(rev "2.0")
+		(company "github.com/AdrianTheHacker")
+	)
 	(text "Debugger"
 		(exclude_from_sim no)
