File: electrical/screen.kicad_sch (KiCad schematic)
At the start: 0 parts

Commit message: Completing schematic.
Parts:
- added C12, C13, C14, C15, C16, C17, C18, C19, C20: 1UF, adrians_favs:SMD_CAPACITOR_CERAMIC_0603, symbol adrians_favs:SMD_CAPACITOR_CERAMIC_0603_1UF
- added D2, D3, D4: SMD_DIODE_MBR0530T1G, adrians_favs:SMD_DIODE_MBR0530T1G, symbol adrians_favs:SMD_DIODE_MBR0530T1G
- added J2: 6871XX149022_687124149022, adrians_favs:SMD_CONNECTOR_RIBBON_CABLE_24_PINS, symbol adrians_favs:SMD_CONNECTOR_RIBBON_CABLE_24_PINS
- added L1: 47uH, adrians_favs:SMD_INDUCTOR_0603, symbol adrians_favs:SMD_INDUCTOR_0603_47UH
- added Q1: SMD_MOSFET_NX3008NBKS, adrians_favs:SMD_MOSFET_NX3008NBKS, symbol adrians_favs:SMD_MOSFET_NX3008NBKS
- added R10: 1KR, adrians_favs:SMD_RESISTOR_0603, symbol adrians_favs:SMD_RESISTOR_0603_1KR
- added R11: 1.5KR, adrians_favs:SMD_RESISTOR_0603, symbol adrians_favs:SMD_RESISTOR_0603_1P5KR
- added R12: 2.2R, adrians_favs:SMD_RESISTOR_0603, symbol adrians_favs:SMD_RESISTOR_0603_2P2R
Connections:
- new net: C18.1, D2.2 (A), L1.1, Q1.6 (D1)
- new net: C18.2, D3.2 (A), D4.1 (K)
- new net +3V0: C15.2, J2.15, J2.16, L1.2, R10.1
- new net 1V8: C16.2, J2.18, R10.2, R11.2
- new net EINK_BUSY: J2.9
- new net EINK_CS: J2.12
- new net EINK_D_C: J2.11
- new net EINK_RST: J2.10
- new net EINK_SCL: J2.13
- new net EINK_SDA: J2.14
- new net GDR: J2.2, Q1.2 (G1), R12.2
- new net GND: C12.1, C13.1, C14.1, C15.1, C16.1, C17.1, C19.2, C20.1, D3.1 (K), J2.17, J2.6, J2.7, J2.8, R11.1
- new net RESE: J2.3, Q1.1 (S1), R12.1
- new net VCOM: C13.2, J2.24
- new net VGH: C20.2, D2.1 (K), J2.21
- new net VGL: C19.1, D4.2 (A), J2.23
- new net VSH1: C17.2, J2.20
- new net VSH2: C14.2, J2.5
- new net VSL: C12.2, J2.22
- no-connect marks 0 -> 8

Commit message: Completing PCB layout.
Connections:
- net GND: now also C12.2, C13.2; no longer C12.1, C13.1
- net VCOM: now also C13.1; no longer C13.2
- net VSL: now also C12.1; no longer C12.2
Other:
- moved on the sheet: C12, C13
Changed lines of the file:
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@@
 	(symbol
 		(lib_id "adrians_favs:SMD_CAPACITOR_CERAMIC_0603_1UF")
-		(at 53.34 167.64 90)
+		(at 53.34 167.64 270)
+		(mirror x)
 		(unit 1)
 		(exclude_from_sim no)
@@
 		)
 		(property "Footprint" "adrians_favs:SMD_CAPACITOR_CERAMIC_0603"
-			(at 57.15 166.6748 0)
+			(at 49.53 166.6748 0)
 			(effects
 				(font
@@
 	(symbol
 		(lib_id "adrians_favs:SMD_CAPACITOR_CERAMIC_0603_1UF")
-		(at 53.34 154.94 90)
+		(at 53.34 154.94 270)
+		(mirror x)
 		(unit 1)
 		(exclude_from_sim no)
@@
 		)
 		(property "Footprint" "adrians_favs:SMD_CAPACITOR_CERAMIC_0603"
-			(at 57.15 153.9748 0)
-			(effects
-				(font
+			(at 49.53 153.9748 0)
+			(effects
+				(font

Commit message: Adding manufacturer and manufacturer number to path.
Parts:
- C12, C13, C14, C15, C16, C17, C18, C19, C20: MFG (none) -> KYOCERA AVX; MFG P/N (none) -> 0603DC105MAT2A
- D2, D3, D4: MFG (none) -> onsemi; MFG P/N (none) -> MBR0530T1G
- J2: MFG (none) -> Würth Elektronik; MFG P/N (none) -> 687124149022
- L1: MFG (none) -> TAIYO YUDEN; MFG P/N (none) -> LBMF1608T470K
- Q1: MFG (none) -> Nexperia; MFG P/N (none) -> NX3008NBKS,115
- R10: MFG (none) -> YAGEO; MFG P/N (none) -> SR0603JR-071KL
- R11: MFG (none) -> TE Connectivity / Holsworthy; MFG P/N (none) -> RT73F1J1K5BTD
- R12: MFG (none) -> TE Connectivity / Holsworthy; MFG P/N (none) -> CRG0603F2R2

Commit message: Updating schematic pages.
Other:
- company: (none) -> github.com/AdrianTheHacker
- title: (none) -> Etchasketch E-Ink Screen
Changed lines of the file:
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@@
 	(generator_version "9.0")
 	(paper "A4")
+	(title_block
+		(title "Etchasketch E-Ink Screen")
+		(rev "2.0")
+		(company "github.com/AdrianTheHacker")
+	)
 	(bus_alias "EINK_INTERFACE"
 		(members "EINK_SDA" "EINK_SCL" "EINK_CS" "EINK_D_C" "EINK_RST" "EINK_BUSY")
