File: electrical/user_input.kicad_sch (KiCad schematic)
At the start: 0 parts

Commit message: Adding user input.
Parts:
- added R7, R8: 10KR, adrians_favs:SMD_RESISTOR_0603, symbol adrians_favs:SMD_RESISTOR_0603_10KR
- added RV1, RV2: 100KR, adrians_favs:THT_POTENTIOMETER_100KR, symbol adrians_favs:THT_POTENTIOMETER_100KR
- added SW3, SW4: SMD_BUTTON, adrians_favs:SMD_BUTTON, symbol adrians_favs:SMD_BUTTON
Connections:
- new net +3V0: R7.2, R8.2, RV1.3, RV2.3
- new net BUTTON_1: R7.1, SW3.3 (K), SW3.4 (A)
- new net BUTTON_2: R8.1, SW4.3 (K), SW4.4 (A)
- new net GND: RV1.2, RV2.2, SW3.1, SW3.2, SW4.1, SW4.2
- new net POT_1: RV1.1
- new net POT_2: RV2.1

Commit message: Adding manufacturer and manufacturer number to path.
Parts:
- R7, R8: MFG (none) -> Vishay / Draloric; MFG P/N (none) -> RCA060310K0JNEA
- RV1, RV2: MFG (none) -> TT Electronics/BI; MFG P/N (none) -> P0915N-FC15BR100K
- SW3, SW4: MFG (none) -> E-Switch; MFG P/N (none) -> TL3301CF260QG; Store (none) -> https://mou.sr/3MCeAPf
Changed lines of the file:
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@@
 	)
 	(symbol
+		(lib_name "SMD_BUTTON_1")
 		(lib_id "adrians_favs:SMD_BUTTON")
 		(at 119.38 73.66 0)
@@
 			)
 		)
+		(property "MFG" "E-Switch"
+			(at 119.38 73.66 0)
+			(effects
+				(font
+					(size 1.27 1.27)
+				)
+				(hide yes)
+			)
+		)
+		(property "MFG P/N" "TL3301CF260QG"
+			(at 119.38 73.66 0)
+			(effects
+				(font
+					(size 1.27 1.27)
+				)
+				(hide yes)
+			)
+		)
+		(property "https://mou.sr/3MG6oNW" ""
+			(at 119.38 73.66 0)
+			(effects
+				(font
+					(size 1.27 1.27)
+				)
+				(hide yes)
+			)
+		)
+		(property "Store" "https://mou.sr/3MCeAPf"
+			(at 119.38 73.66 0)
+			(effects
+				(font
+					(size 1.27 1.27)
+				)
+				(hide yes)
+			)
+		)
 		(pin "3"
 		)
@@
 			)
 		)
+		(property "MFG" "TT Electronics/BI"
+			(at 151.13 107.95 0)
+			(effects
+				(font
+					(size 1.27 1.27)
+				)
+				(hide yes)
+			)
+		)
+		(property "MFG P/N" "P0915N-FC15BR100K"
+			(at 151.13 107.95 0)
+			(effects
+				(font
+					(size 1.27 1.27)
+				)
+				(hide yes)
+			)
+		)
+		(property "https://mou.sr/3MG6oNW" ""
+			(at 151.13 107.95 0)
+			(effects
+				(font
+					(size 1.27 1.27)
+				)
+				(hide yes)
+			)
+		)
 		(pin "3"
 		)
@@
 			)
 		)
+		(property "MFG" "TT Electronics/BI"
+			(at 107.95 107.95 0)
+			(effects
+				(font
+					(size 1.27 1.27)
+				)
+				(hide yes)
+			)
+		)
+		(property "MFG P/N" "P0915N-FC15BR100K"
+			(at 107.95 107.95 0)
+			(effects
+				(font
+					(size 1.27 1.27)
+				)
+				(hide yes)
+			)
+		)
+		(property "https://mou.sr/3MG6oNW" ""
+			(at 107.95 107.95 0)
+			(effects
+				(font
+					(size 1.27 1.27)
+				)
+				(hide yes)
+			)
+		)
 		(pin "3"
 		)
@@
 			)
 		)
+		(property "MFG" "Vishay / Draloric"
+			(at 146.05 71.12 0)
+			(effects
+				(font
+					(size 1.27 1.27)
+				)
+				(hide yes)
+			)
+		)
+		(property "MFG P/N" "RCA060310K0JNEA"
+			(at 146.05 71.12 0)
+			(effects
+				(font
+					(size 1.27 1.27)
+				)
+				(hide yes)
+			)
+		)
+		(property "https://mou.sr/3MG6oNW" ""
+			(at 146.05 71.12 0)
+			(effects
+				(font
+					(size 1.27 1.27)
+				)
+				(hide yes)
+			)
+		)
 		(pin "1"
 		)
@@
 			)
 		)
+		(property "MFG" "E-Switch"
+			(at 119.38 88.9 0)
+			(effects
+				(font
+					(size 1.27 1.27)
+				)
+				(hide yes)
+			)
+		)
+		(property "MFG P/N" "TL3301CF260QG"
+			(at 119.38 88.9 0)
+			(effects
+				(font
+					(size 1.27 1.27)
+				)
+				(hide yes)
+			)
+		)
+		(property "https://mou.sr/3MG6oNW" ""
+			(at 119.38 88.9 0)
+			(effects
+				(font
+					(size 1.27 1.27)
+				)
+				(hide yes)
+			)
+		)
+		(property "Store" "https://mou.sr/3MCeAPf"
+			(at 119.38 88.9 0)
+			(effects
+				(font
+					(size 1.27 1.27)
+				)
+				(hide yes)
+			)
+		)
 		(pin "3"
 		)
@@
 			(at 146.05 86.36 0)
 			(effects
+				(font
+					(size 1.27 1.27)
+				)
+				(hide yes)
+			)
+		)
+		(property "MFG" "Vishay / Draloric"
+			(at 146.05 86.36 0)
+			(effects
+				(font
+					(size 1.27 1.27)
+				)
+				(hide yes)
+			)
+		)
+		(property "MFG P/N" "RCA060310K0JNEA"
+			(at 146.05 86.36 0)
+			(effects
+				(font
+					(size 1.27 1.27)
+				)
+				(hide yes)
+			)
+		)
+		(property "https://mou.sr/3MG6oNW" ""
+			(at 146.05 86.36 0)
+			(effects

Commit message: Updating schematic pages.
Other:
- company: (none) -> github.com/AdrianTheHacker
- title: (none) -> Etchasketch User Interface
Changed lines of the file:
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@@
 	(generator_version "9.0")
 	(paper "A4")
+	(title_block
+		(title "Etchasketch User Interface")
+		(date "2025-12-12")
+		(rev "2.0")
+		(company "github.com/AdrianTheHacker")
+	)
 	(bus_alias "USER_INPUTS"
 		(members "BUTTON_1" "BUTTON_2" "POT_1" "POT_2")
