File: electrical/wifi.kicad_sch (KiCad schematic)
At the start: 2 parts

Commit message: Adding user input.
Changed lines of the file:
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@@
 	)
 	(global_label "GND"
-		(shape input)
+		(shape passive)
 		(at 38.1 30.48 180)
 		(fields_autoplaced yes)
@@
 		)
 		(property "Intersheetrefs" "${INTERSHEET_REFS}"
-			(at 31.2443 30.48 0)
+			(at 32.3556 30.48 0)
 			(effects
 				(font
@@
 	)
 	(global_label "+3V0"
-		(shape input)
+		(shape passive)
 		(at 38.1 24.13 180)
 		(fields_autoplaced yes)
@@
 		)
 		(property "Intersheetrefs" "${INTERSHEET_REFS}"
-			(at 30.0348 24.13 0)
+			(at 31.1461 24.13 0)
 			(effects
 				(font

Commit message: Improving manufacturability of the board.
Parts:
- IC2: now not fitted; now left out of the parts list
Changed lines of the file:
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@@
 		(unit 1)
 		(exclude_from_sim no)
-		(in_bom yes)
+		(in_bom no)
 		(on_board yes)
-		(dnp no)
+		(dnp yes)
 		(fields_autoplaced yes)
 		(property "Reference" "IC2"

Commit message: Adding manufacturer and manufacturer number to path.
Parts:
- IC2: MFG (none) -> Adafruit; MFG P/N (none) -> 4201
- R6: MFG (none) -> Vishay / Draloric; MFG P/N (none) -> RCA060310K0JNEA
Changed lines of the file:
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@@
+			)
+		)
+		(property "MFG" "Adafruit"
+			(at 184.15 85.09 90)
+			(effects
+				(font
+					(size 1.27 1.27)
+				)
+				(hide yes)
+			)
+		)
+		(property "MFG P/N" "4201"
+			(at 184.15 85.09 90)
+			(effects
+				(font
+					(size 1.27 1.27)
+				)
+				(hide yes)
+			)
+		)
+		(property "https://mou.sr/3MG6oNW" ""
+			(at 184.15 85.09 90)
+			(effects
+				(font
+					(size 1.27 1.27)
+				)
+				(hide yes)
 			)
 		)
@@
 			(effects
 				(font
+					(size 1.27 1.27)
+				)
+				(hide yes)
+			)
+		)
+		(property "MFG" "Vishay / Draloric"
+			(at 160.02 111.76 90)
+			(effects
+				(font
+					(size 1.27 1.27)
+				)
+				(hide yes)
+			)
+		)
+		(property "MFG P/N" "RCA060310K0JNEA"
+			(at 160.02 111.76 90)
+			(effects
+				(font
+					(size 1.27 1.27)
+				)
+				(hide yes)
+			)
+		)
+		(property "https://mou.sr/3MG6oNW" ""
+			(at 160.02 111.76 90)
+			(effects
+				(font

Commit message: Updating schematic pages.
Other:
- company: (none) -> github.com/AdrianTheHacker
- title: (none) -> Etchasketch WiFi Module Interface
Changed lines of the file:
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@@
 	(generator_version "9.0")
 	(paper "A4")
+	(title_block
+		(title "Etchasketch WiFi Module Interface")
+		(rev "2.0")
+		(company "github.com/AdrianTheHacker")
+	)
 	(bus_alias "WIFI_INTERFACE"
 		(members "WIFI_SCK" "WIFI_MISO" "WIFI_MOSI" "WIFI_CS" "WIFI_BUSY" "WIFI_RESET")
